Commit message: Hopefully the final commit to the repo so its ready for everyone yaygit add .!

File: configs/warthog.urdf.xacro (robot description, xacro)
@@ -1,5 +1,4 @@
-<?xml version="1.0"?>
+<?xml version='1.0'?>
 <robot name="warthog" xmlns:xacro="http://www.ros.org/wiki/xacro">
-  <!-- Basic properties -->
   <xacro:property name="PI" value="3.1415926535897931"/>
   <xacro:property name="wheel_radius" value="0.3" />
@@ -22,5 +21,12 @@
   <xacro:property name="chassis_mass" value="100" />
   <xacro:property name="dummy_inertia" value="1e-09"/>
-  <!-- Optional paint colors -->
+  <!--
+    Optional paint colors.
+    Available colors:
+      - yellow (default)
+      - orange
+      - olive
+      - sand
+  -->
   <xacro:property name="warthog_color" value="$(optenv WARTHOG_COLOR yellow)" />
   <xacro:if value="${warthog_color == 'yellow'}">
@@ -36,5 +42,4 @@
     <xacro:property name="warthog_color_rgba" value="0.86 0.75 0.54 1.0" />
   </xacro:if>
-  <!-- Inertia macros -->
   <xacro:macro name="wheel_inertia" params="m r h">
     <inertia ixx="${m*(3*r*r+h*h)/12}" ixy="0" ixz="0"
@@ -47,5 +52,4 @@
              izz="${m*(x*x+z*z)/12}" />
   </xacro:macro>
-  <!-- Materials -->
   <material name="dark_grey"><color rgba="0.2 0.2 0.2 1.0" /></material>
   <material name="light_grey"><color rgba="0.4 0.4 0.4 1.0" /></material>
@@ -54,5 +58,4 @@
   <material name="white"><color rgba="0.9 0.9 0.9 1.0" /></material>
   <material name="red"><color rgba="0.9 0.0 0.0 1.0" /></material>
-  <!-- Wheel macro from File #2 (includes collision) -->
   <xacro:macro name="wheel" params="prefix side *joint_pose">
     <link name="${prefix}_${side}_wheel_link">
@@ -102,5 +105,4 @@
     </transmission>
   </xacro:macro>
-  <!-- Track macro from File #2 (includes collision geometry) -->
   <xacro:macro name="track" params="prefix side *joint_pose">
     <link name="${prefix}_${side}_track_link">
@@ -125,5 +127,5 @@
       <axis xyz="0 1 0"/>
     </joint>
-    <!-- This adds wheels that rotate instead of tracks -->
+    <!-- This adds wheels that rotate instead of tracks. -->
     <link name="${prefix}_${side}_wheel_link">
       <collision>
@@ -151,5 +153,32 @@
     </transmission>
   </xacro:macro>
-  <!-- Diff Unit Macro from File #2 -->
+  <xacro:unless value="$(optenv WARTHOG_TRACKS 0)">
+    <xacro:wheel prefix="front" side="left">
+      <origin xyz="${axle_x_offset*1} ${axle_y_offset*1} ${axle_z_offset}" rpy="0 0 0" />
+    </xacro:wheel>
+    <xacro:wheel prefix="front" side="right">
+      <origin xyz="${axle_x_offset*1} ${axle_y_offset*-1} ${axle_z_offset}" rpy="0 0 0" />
+    </xacro:wheel>
+    <xacro:wheel prefix="rear" side="left">
+      <origin xyz="${axle_x_offset*-1} ${axle_y_offset*1} ${axle_z_offset}" rpy="0 0 0" />
+    </xacro:wheel>
+    <xacro:wheel prefix="rear" side="right">
+      <origin xyz="${axle_x_offset*-1} ${axle_y_offset*-1} ${axle_z_offset}" rpy="0 0 0" />
+    </xacro:wheel>
+  </xacro:unless>
+  <xacro:if value="$(optenv WARTHOG_TRACKS 0)">
+    <xacro:track prefix="front" side="left">
+      <origin xyz="${axle_x_offset*1} ${axle_y_offset*1} ${axle_z_offset}" rpy="0 0 0" />
+    </xacro:track>
+    <xacro:track prefix="front" side="right">
+      <origin xyz="${axle_x_offset*1} ${axle_y_offset*-1} ${axle_z_offset}" rpy="0 0 0" />
+    </xacro:track>
+    <xacro:track prefix="rear" side="left">
+      <origin xyz="${axle_x_offset*-1} ${axle_y_offset*1} ${axle_z_offset}" rpy="0 0 ${PI}" />
+    </xacro:track>
+    <xacro:track prefix="rear" side="right">
+      <origin xyz="${axle_x_offset*-1} ${axle_y_offset*-1} ${axle_z_offset}" rpy="0 0 ${PI}" />
+    </xacro:track>
+  </xacro:if>
   <xacro:macro name="diff_unit" params="prefix side left">
     <link name="${prefix}_diff_unit_link">
@@ -208,4 +237,5 @@
         <geometry>
           <cylinder radius="0.0205" length="0.014"/>
+          <material name="red"><color rgba="0.9 0.0 0.0 1.0" /></material>
         </geometry>
       </collision>
@@ -214,4 +244,5 @@
         <geometry>
           <cylinder radius="0.0205" length="0.014"/>
+          <material name="red"><color rgba="0.9 0.0 0.0 1.0" /></material>
         </geometry>
       </collision>
@@ -241,5 +272,5 @@
       <origin xyz="0 0 0" rpy="0 0 ${side*PI/2}"/>
       <parent link="${prefix}_diff_unit_link" />
-      <child link="${prefix}_diff_unit_antenna_link"/>
+      <child link="${prefix}_diff_unit_antenna_link" />
     </joint>
     <!-- E-stop Antenna -->
@@ -284,5 +315,5 @@
     <joint name="${prefix}_diff_unit_headlight_joint" type="fixed">
       <parent link="${prefix}_diff_unit_link" />
-      <child link="${prefix}_diff_unit_headlight_link"/>
+      <child link="${prefix}_diff_unit_headlight_link" />
       <origin xyz="0 0 0" rpy="0 0 0"/>
     </joint>
@@ -315,5 +346,5 @@
     <joint name="${prefix}_diff_unit_taillight_joint" type="fixed">
       <parent link="${prefix}_diff_unit_link" />
-      <child link="${prefix}_diff_unit_taillight_link"/>
+      <child link="${prefix}_diff_unit_taillight_link" />
       <origin xyz="0 0 0" rpy="0 0 0"/>
     </joint>
@@ -340,5 +371,12 @@
     </gazebo>
   </xacro:macro>
-  <!-- Chassis link from File #2 -->
+  <xacro:diff_unit prefix="left" side="1" left="true"/>
+  <xacro:diff_unit prefix="right" side="-1" left="false"/>
+  <link name="base_link"></link>
+  <joint name="base_link_joint" type="fixed">
+    <origin xyz="0 0 0.025" rpy="0 0 0" />
+    <parent link="base_link"/>
+    <child link="chassis_link" />
+  </joint>
   <link name="chassis_link">
     <inertial>
@@ -355,4 +393,11 @@
       <material name="black"><color rgba="0.15 0.15 0.15 1.0" /></material>
     </visual>
+    <visual>
+      <origin xyz="0 0 0" rpy="0 0 0"/>
+      <geometry>
+        <mesh filename="package://warthog_description/meshes/e-stop.stl" />
+      </geometry>
+      <material name="red"><color rgba="0.9 0.0 0.0 1.0" /></material>
+    </visual>
     <collision>
       <origin xyz="0 0 0" rpy="0 0 0"/>
@@ -362,5 +407,4 @@
     </collision>
   </link>
-  <!-- POV Camera (from File #2) -->
   <link name="camera_link">
     <inertial>
@@ -372,5 +416,5 @@
     <parent link="chassis_link"/>
     <child link="camera_link"/>
-    <origin xyz="-3 0 3" rpy="0 0.485 0"/>
+    <origin xyz="-3 0 3" rpy="0 0.485 0"/> <!-- 3m behind and 2m above the chassis -->
   </joint>
   <gazebo reference="camera_link">
@@ -378,5 +422,5 @@
       <update_rate>30.0</update_rate>
       <camera>
-        <horizontal_fov>1.396</horizontal_fov>
+        <horizontal_fov>1.396</horizontal_fov> <!-- Field of View -->
         <image>
           <width>1920</width>
@@ -393,6 +437,5 @@
     </sensor>
   </gazebo>
-  <!-- Additional structure from File #2 -->
-  <link name="top_chassis_link"/>
+  <link name="top_chassis_link"></link>
   <joint name="top_link_joint" type="fixed">
     <origin xyz="0 0 0.27218" rpy="0 0 0" />
@@ -400,4 +443,5 @@
     <child link="top_chassis_link" />
   </joint>
+  <!-- This link is purely to complete the visual look -->
   <link name="diff_link">
     <visual>
@@ -428,54 +472,27 @@
     <origin xyz="-0.5826 0 0.24979" rpy="0 0 0" />
   </joint>
-  <link name="imu_link"/>
+  <link name="imu_link" />
   <joint name="imu_link_joint" type="fixed">
     <origin xyz="$(optenv WARTHOG_IMU_XYZ 0 0 0)" rpy="$(optenv WARTHOG_IMU_RPY 0 0 0)" />
     <parent link="chassis_link"/>
-    <child link="imu_link"/>
+    <child link="imu_link" />
   </joint>
-  <!-- Bring in simulation data and accessories -->
+  <!-- Bring in simulation data for Gazebo. -->
   <xacro:include filename="$(find warthog_description)/urdf/warthog.gazebo" />
+  <!-- Optional standard accessories, including their simulation data. The rendering
+       of these into the final description is controlled by optenv variables, which
+       default each one to off.-->
   <xacro:include filename="$(find warthog_description)/urdf/accessories.urdf.xacro" />
-  <!-- OutdoorNav arguments and optional config -->
-  <xacro:arg name="outdoornav_enabled" default="$(optenv OUTDOORNAV_ENABLED 0)" />
+  <!-- OutdoorNav -->
+  <xacro:arg name="outdoornav_enabled"       default="$(optenv OUTDOORNAV_ENABLED 0)" />
   <xacro:arg name="outdoornav_configuration" default="$(optenv OUTDOORNAV_CONFIGURATION standard)" />
+  <!-- OutdoorNav URDF Config -->
   <xacro:if value="$(arg outdoornav_enabled)">
     <xacro:include filename="$(find cpr_onav_description)/urdf/outdoornav_description.urdf.xacro" />
     <xacro:outdoornav_sensors outdoornav_configuration="$(arg outdoornav_configuration)" />
   </xacro:if>
-  <!-- Optional custom includes -->
+  <!-- Optional custom includes. -->
   <xacro:include filename="$(optenv WARTHOG_URDF_EXTRAS empty.urdf)" />
+  <!-- Optional for Clearpath internal softwares -->
   <xacro:include filename="$(optenv CPR_URDF_EXTRAS empty.urdf)" />
-  <!-- Ruler (from File #1; purely visual) -->
-  <link name="ruler_link">
-    <inertial>
-      <origin xyz="0 0 0" rpy="0 0 0"/>
-      <mass value="0.001"/>
-      <inertia ixx="1e-06" ixy="0" ixz="0" iyy="1e-06" iyz="0" izz="1e-06"/>
-    </inertial>
-    <visual>
-      <origin xyz="0 0 0" rpy="0 0 0"/>
-      <geometry>
-        <mesh filename="package://warthog_description/meshes/RULER.dae" scale="1 1 1"/>
-      </geometry>
-    </visual>
-  </link>
-  <joint name="ruler_joint" type="fixed">
-    <parent link="rear_right_wheel_link"/>
-    <child link="ruler_link"/>
-    <origin xyz="0 0 0" rpy="0 0 0"/>
-  </joint>
-  <gazebo reference="ruler_link">
-    <selfCollide>false</selfCollide>
-    <contact>
-      <bitmask>0</bitmask>
-    </contact>
-  </gazebo>
-  <gazebo>
-    <static>true</static>
-    <selfCollide>false</selfCollide>
-    <contact>
-      <bitmask>0</bitmask>
-    </contact>
-  </gazebo>
-</robot>
+  </robot>
